File: Hardware/SparkFun_GNSS_HAT+.kicad_sch (KiCad schematic)
At the start: 81 parts, among them J1 Raspberry_Pi_2x20_SMD_Passthr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, J2 Conn_02x10, J3 U.FL, J4 Conn_02x10, J5 microSD, J6 USB_C_Receptacle, J7 SMA_Edge, J8 Qwiic_RA, U1 CAT24C512WI-GT3, U2 AP7361C-3.3V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

Commit message: More WIP
Parts:
- removed J5: microSD, SparkFun-Connector:microSD_External_Pin, symbol SparkFun-Connector:microSD_PushPush
- removed J8: Qwiic_RA, SparkFun-Connector:JST_SMD_1.0mm-4_RA, symbol SparkFun-Connector:Qwiic_Right_Angle
- removed JP10, JP11, JP12, JP13, JP14, JP15, JP16, JP17, JP18, JP19, JP20, JP21, JP4, JP5, JP6, JP7: Measure, SparkFun-Jumper:Jumper_2_PTH_SMD_Combo-NC, symbol SparkFun-Jumper:Jumper_Measure
- added J5: microSD_Friction, SparkFun-Connector:microSD_Friction_Fit_Common, symbol SparkFun-Connector:microSD_Friction
- added J8: Qwiic_Vertical, SparkFun-Connector:JST_SMD_1.0mm-4_Vertical, symbol SparkFun-Connector:Qwiic_Vertical
- added JP10, JP11, JP12, JP13, JP14, JP15, JP16, JP17, JP18, JP19, JP20, JP21, JP4, JP5, JP6, JP7: ~, SparkFun-Jumper:Jumper_2_NC_Trace, symbol SparkFun-Jumper:SolderJumper_2_Bridged
- added ST1, ST2, ST3, ST4: Standoff, SparkFun-Hardware:Standoff, symbol SparkFun-Hardware:Standoff
Connections:
- net 3.3V: now also J5.4 (VDD), J8.2 (Pin_2)
- net CTS2: now also JP17.2 (B)
- net CTS3: now also JP13.2 (B)
- net EVENTA: now also JP8.1 (A)
- net EVENTB: now also JP9.1 (A)
- net GND: now also J5.10 (SHIELD), J5.6 (VSS), J8.1 (Pin_1)
- net PPS1: now also JP22.1 (A), JP6.1 (A); no longer JP22.2 (B)
- net PPS2: now also JP7.1 (A)
- net PVT_LED: now also JP21.1 (A); no longer JP9.2 (B)
- net RTK_LED: now also JP20.1 (A); no longer JP8.2 (B)
- net RTS2: now also JP16.2 (B)
- net RTS3: now also JP12.2 (B)
- net RXD1: now also JP4.1 (A)
- net RXD2: now also JP14.2 (B)
- net RXD3: now also JP10.2 (B)
- net RXD4: now also JP18.2 (B)
- net SCL: now also J8.4 (Pin_4)
- net SDA: now also J8.3 (Pin_3)
- net SD_CLK: now also J5.5 (CLK/SCK)
- net SD_CMD: now also J5.3 (CMD/SDI)
- net SD_DAT0: now also J5.7 (DAT0/SDO)
- net SD_DAT3: now also J5.2 (DAT3/~{CS})
- net TXD1: now also JP5.1 (A)
- net TXD2: now also JP15.2 (B)
- net TXD3: now also JP11.2 (B)
- net TXD4: now also JP19.2 (B)
- net at J1.15 (GPIO22): now also JP6.2 (B)
- net at J1.23 (SCLK0/GPIO11): now also JP17.1 (A)
- net at J1.16 (GPIO23): now also JP7.2 (B)
- net at R12.2: now also JP21.2 (B); no longer JP9.1 (A)
- net at R11.2: now also JP20.2 (B); no longer JP8.1 (A)
- net at J1.24 (~{CE0}/GPIO8): now also JP14.1 (A)
- net at J1.26 (~{CE1}/GPIO7): now also JP13.1 (A)
- net at J1.33 (PWM1/GPIO13): now also JP19.1 (A)
- net at J1.31 (GCLK2/GPIO6): now also JP12.1 (A)
- net at J1.29 (GCLK1/GPIO5): now also JP11.1 (A)
- net at J1.8 (GPIO14/TXD): now also JP4.2 (B)
- net at R13.2: now also JP22.2 (B); no longer JP22.1 (A)
- net at J1.18 (GPIO24): now also JP8.2 (B)
- net at J1.19 (PICO0/GPIO10): now also JP16.1 (A)
- net at J1.21 (POCI0/GPIO9): now also JP15.1 (A)
- net at J1.7 (GCLK0/GPIO4): now also JP10.1 (A)
- net at J1.32 (PWM0/GPIO12): now also JP18.1 (A)
- net at J1.22 (GPIO25): now also JP9.2 (B)
- net at J1.10 (GPIO15/RXD): now also JP5.2 (B)
- new net: J8.NC1 (NC), J8.NC2 (NC)

Commit message: More WIP
Parts:
- removed H1, H2, H3, H4: MountingHole, MountingHole:MountingHole_2.7mm_M2.5_DIN965, symbol Mechanical:MountingHole
- added ST5, ST6, ST7, ST8: Standoff, SparkFun-Hardware:Standoff_Raspberry-Pi_HAT+, symbol SparkFun-Hardware:Standoff_Raspberry-Pi_HAT+
- J2, J4: PROD_ID (none) -> CONN-22476
Connections:
- net D+: now also TR1.4; no longer TR1.2
- net D-: now also TR1.2; no longer TR1.4
- net at D1.1 (I/O1), J6.A6 (D+), J6.B6 (D+): now also TR1.3; no longer TR1.1
- net at D1.3 (I/O2), J6.A7 (D-), J6.B7 (D-): now also TR1.1; no longer TR1.3

Commit message: Routed
Connections:
- net SD_CLK: now also D2.3 (K2); no longer D2.4 (K3)
- net SD_CMD: now also D2.4 (K3); no longer D2.5 (K4)
- net SD_DAT0: now also D2.1 (K1); no longer D2.3 (K2)
- net SD_DAT3: now also D2.5 (K4); no longer D2.1 (K1)
Changed lines of the file:
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@@
+	)
+	(junction
+		(at 67.31 171.45)
+		(diameter 0)
+		(color 0 0 0 0)
 	)
 	(junction
@@
 	)
 	(junction
-		(at 62.23 173.99)
-		(diameter 0)
-		(color 0 0 0 0)
-	)
-	(junction
-		(at 59.69 176.53)
-		(diameter 0)
-		(color 0 0 0 0)
-	)
-	(junction
-		(at 64.77 171.45)
+		(at 59.69 163.83)
 		(diameter 0)
 		(color 0 0 0 0)
@@
 	)
 	(junction
+		(at 62.23 176.53)
+		(diameter 0)
+		(color 0 0 0 0)
+	)
+	(junction
 		(at 54.61 153.67)
 		(diameter 0)
@@
 	)
 	(junction
-		(at 67.31 163.83)
+		(at 64.77 173.99)
 		(diameter 0)
 		(color 0 0 0 0)
@@
 	(wire
 		(pts
-			(xy 67.31 163.83) (xy 67.31 179.07)
-		)
-		(stroke
-			(width 0)
-			(type default)
-		)
-	)
-	(wire
-		(pts
 			(xy 175.26 27.94) (xy 175.26 29.21)
 		)
@@
 	(wire
 		(pts
+			(xy 64.77 173.99) (xy 64.77 179.07)
+		)
+		(stroke
+			(width 0)
+			(type default)
+		)
+	)
+	(wire
+		(pts
 			(xy 234.95 68.58) (xy 234.95 74.93)
 		)
@@
 	(wire
 		(pts
+			(xy 62.23 176.53) (xy 62.23 179.07)
+		)
+		(stroke
+			(width 0)
+			(type default)
+		)
+	)
+	(wire
+		(pts
 			(xy 219.71 111.76) (xy 219.71 113.03)
 		)
@@
 	(wire
 		(pts
-			(xy 62.23 173.99) (xy 62.23 179.07)
-		)
-		(stroke
-			(width 0)
-			(type default)
-		)
-	)
-	(wire
-		(pts
 			(xy 118.11 36.83) (xy 120.65 36.83)
 		)
@@
 	(wire
 		(pts
-			(xy 64.77 171.45) (xy 64.77 179.07)
-		)
-		(stroke
-			(width 0)
-			(type default)
-		)
-	)
-	(wire
-		(pts
-			(xy 59.69 176.53) (xy 59.69 179.07)
-		)
-		(stroke
-			(width 0)
-			(type default)
-		)
-	)
-	(wire
-		(pts
 			(xy 76.2 45.72) (xy 77.47 45.72)
 		)
@@
 	(wire
 		(pts
-			(xy 59.69 176.53) (xy 72.39 176.53)
-		)
-		(stroke
-			(width 0)
-			(type default)
-		)
-	)
-	(wire
-		(pts
 			(xy 237.49 39.37) (xy 238.76 39.37)
 		)
@@
 	(wire
 		(pts
+			(xy 59.69 163.83) (xy 62.23 163.83)
+		)
+		(stroke
+			(width 0)
+			(type default)
+		)
+	)
+	(wire
+		(pts
 			(xy 204.47 34.29) (xy 207.01 34.29)
 		)
@@
 	(wire
 		(pts
+			(xy 64.77 173.99) (xy 72.39 173.99)
+		)
+		(stroke
+			(width 0)
+			(type default)
+		)
+	)
+	(wire
+		(pts
 			(xy 173.99 46.99) (xy 176.53 46.99)
 		)
@@
 	(wire
 		(pts
-			(xy 62.23 173.99) (xy 72.39 173.99)
-		)
-		(stroke
-			(width 0)
-			(type default)
-		)
-	)
-	(wire
-		(pts
 			(xy 218.44 113.03) (xy 219.71 113.03)
 		)
@@
 	(wire
 		(pts
-			(xy 64.77 171.45) (xy 72.39 171.45)
-		)
-		(stroke
-			(width 0)
-			(type default)
-		)
-	)
-	(wire
-		(pts
 			(xy 180.34 138.43) (xy 180.34 139.7)
 		)
@@
 	(wire
 		(pts
+			(xy 67.31 171.45) (xy 67.31 179.07)
+		)
+		(stroke
+			(width 0)
+			(type default)
+		)
+	)
+	(wire
+		(pts
 			(xy 76.2 40.64) (xy 77.47 40.64)
 		)
@@
 	(wire
 		(pts
-			(xy 62.23 163.83) (xy 67.31 163.83)
-		)
-		(stroke
-			(width 0)
-			(type default)
-		)
-	)
-	(wire
-		(pts
 			(xy 119.38 114.3) (xy 119.38 119.38)
 		)
@@
 	(wire
 		(pts
-			(xy 67.31 163.83) (xy 72.39 163.83)
-		)
-		(stroke
-			(width 0)
-			(type default)
-		)
-	)
-	(wire
-		(pts
-			(xy 52.07 171.45) (xy 64.77 171.45)
+			(xy 62.23 163.83) (xy 72.39 163.83)
+		)
+		(stroke
+			(width 0)
+			(type default)
+		)
+	)
+	(wire
+		(pts
+			(xy 52.07 171.45) (xy 67.31 171.45)
 		)
 		(stroke
@@
 	(wire
 		(pts
+			(xy 67.31 171.45) (xy 72.39 171.45)
+		)
+		(stroke
+			(width 0)
+			(type default)
+		)
+	)
+	(wire
+		(pts
 			(xy 224.79 139.7) (xy 224.79 140.97)
 		)
@@
 	(wire
 		(pts
-			(xy 50.8 163.83) (xy 62.23 163.83)
+			(xy 50.8 163.83) (xy 59.69 163.83)
 		)
 		(stroke
@@
 	(wire
 		(pts
-			(xy 50.8 173.99) (xy 62.23 173.99)
+			(xy 50.8 173.99) (xy 64.77 173.99)
 		)
 		(stroke
@@
 		)
 	)
+	(wire
+		(pts
+			(xy 62.23 176.53) (xy 72.39 176.53)
+		)
+		(stroke
+			(width 0)
+			(type default)
+		)
+	)
 	(polyline
 		(pts
@@
 	(wire
 		(pts
-			(xy 54.61 176.53) (xy 59.69 176.53)
+			(xy 54.61 176.53) (xy 62.23 176.53)
 		)
 		(stroke
@@
 		)
 		(stroke
+			(width 0)
+			(type default)
+		)
+	)
+	(wire
+		(pts
+			(xy 59.69 163.83) (xy 59.69 179.07)
+		)
+		(stroke

Commit message: Panelized
Changed lines of the file:
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@@
 	(symbol
 		(lib_id "SparkFun-Aesthetic:SparkPNT_Logo")
-		(at 210.82 179.07 0)
+		(at 191.77 176.53 0)
 		(unit 1)
 		(exclude_from_sim no)
@@
 		(fields_autoplaced yes)
 		(property "Reference" "G1"
-			(at 210.82 174.625 0)
+			(at 191.77 172.085 0)
 			(effects
 				(font
@@
 		)
 		(property "Value" "LOGO"
-			(at 210.82 183.515 0)
+			(at 191.77 180.975 0)
 			(effects
 				(font
@@
 		)
 		(property "Footprint" ""
-			(at 210.82 179.07 0)
+			(at 191.77 176.53 0)
 			(effects
 				(font
@@
 		)
 		(property "Datasheet" ""
-			(at 210.82 179.07 0)
+			(at 191.77 176.53 0)
 			(effects
 				(font
@@
 		)
 		(property "Description" ""
-			(at 210.82 179.07 0)
+			(at 191.77 176.53 0)
 			(effects
 				(font
@@
 					(unit 1)
 				)
+			)
+		)
+	)
+	(symbol
+		(lib_id "SparkFun-Aesthetic:Raspberry_Pi_HAT+_Logo")
+		(at 228.6 176.53 0)
+		(unit 1)
+		(exclude_from_sim no)
+		(in_bom yes)
+		(on_board yes)
+		(dnp no)
+		(fields_autoplaced yes)
+		(property "Reference" "#G1"
+			(at 228.6 171.45 0)
+			(effects
+				(font
+					(size 1.27 1.27)
+				)
+				(hide yes)
+			)
+		)
+		(property "Value" "Raspberry_Pi_HAT+_Logo"
+			(at 228.6 181.61 0)
+			(effects
+				(font
+					(size 1.27 1.27)
+				)
+				(hide yes)
+			)
+		)
+		(property "Footprint" ""
+			(at 228.6 176.53 0)
+			(effects
+				(font
+					(size 1.27 1.27)
+				)
+				(hide yes)
+			)
+		)
+		(property "Datasheet" ""
+			(at 228.6 176.53 0)
+			(effects
+				(font
+					(size 1.27 1.27)
+				)
+				(hide yes)
+			)
+		)
+		(property "Description" ""
+			(at 228.6 176.53 0)
+			(effects
+				(font
+					(size 1.27 1.27)
+				)
+				(hide yes)
+			)
+		)
+		(instances
+			(project ""
+				(path "/e3dd3ae4-244d-4cba-9cca-5d2abf83f29a"
+					(reference "#G1")
+					(unit 1)
+				)
