File: Hardware/SparkFun_GNSS_pHAT.kicad_sch (KiCad schematic)
At the start: 85 parts, among them J1 Raspberry_Pi_2x20_SMD_Passthr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, J2 Conn_02x10, J3 U.FL, J4 Conn_02x10, J5 microSD_Friction, J6 USB_C_Receptacle, J7 SMA_Edge, J8 Qwiic_Vertical, U1 CAT24C512WI-GT3, U2 AP7361C-3.3V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

Commit message: Change name to GNSS pHAT
Parts:
- removed D3, D5: Blue, SparkFun-LED:LED_0603_1608Metric_Blue, symbol SparkFun-LED:LED_Blue_0603
- removed G1: LOGO, symbol SparkFun-Aesthetic:SparkPNT_Logo
- removed JP2: ~, SparkFun-Jumper:Jumper_3_NC-2_Trace, symbol SparkFun-Jumper:SolderJumper_3_Bridged123
- removed R11: 2.2k, SparkFun-Resistor:R_0603_1608Metric, symbol SparkFun-Resistor:2.2k_0603
- added D3: White, SparkFun-LED:LED_0603_1608Metric_White, symbol SparkFun-LED:LED_White_0603
- added D5: Yellow, SparkFun-LED:LED_0603_1608Metric_Yellow, symbol SparkFun-LED:LED_Yellow_0603
- added D6: Red, SparkFun-LED:LED_0603_1608Metric_Red, symbol SparkFun-LED:LED_Red_0603
- added G1: SparkFun_Logo, symbol SparkFun-Aesthetic:SparkFun_Logo
- added GPIO26.1: PTH, SparkFun-Connector:1x01, symbol SparkFun-Connector:TestPoint_PTH
- added JP2: ~, SparkFun-Jumper:Jumper_3_NO, symbol SparkFun-Jumper:SolderJumper_3_Open
- added JP23: ~, SparkFun-Jumper:Jumper_2_NC_Trace, symbol SparkFun-Jumper:SolderJumper_2_Bridged
- added R11, R14: 1k, SparkFun-Resistor:R_0603_1608Metric, symbol SparkFun-Resistor:1k_0603
- U1: now not fitted; now left out of the parts list
Connections:
- net 3.3V: now also JP2.2 (B), JP23.2 (B)
- net GND: now also D3.1 (K), D5.1 (K), D6.1 (K)
- net at R1.2: now also JP2.1 (A)
- net at R2.2: now also JP2.3 (C)
- net at R13.1: now also D5.2 (A)
- net at JP20.2 (B): now also R11.2
- net at J1.37 (GPIO26): now also GPIO26.1.1
- new net: D3.2 (A), R11.1
- new net: D6.2 (A), R14.1
- new net: JP23.1 (A), R14.2
Other:
- note added: "Close jumpers to add pull-ups to bus"
- title: SparkFun GNSS HAT+ -> SparkFun GNSS pHAT
- moved on the sheet: 3V3.1, C1, C2, C3, C4, C5, C6, D1, D4, GND.1, J6, JP20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

Commit message: pHAT routed and panelized
Parts:
- removed 3V3.1, GND.1, GPIO26.1, RST.1, WP.1: PTH, SparkFun-Connector:1x01, symbol SparkFun-Connector:TestPoint_PTH
- added J9: Conn_01x05, SparkFun-Connector:1x05, symbol SparkFun-Connector:Conn_01x05
Connections:
- net 3.3V: now also J9.2 (Pin_2)
- net GND: now also J9.1 (Pin_1)
- net WP: now reaches R3.1, U1.7 (WP)
- net WP: now also J9.3 (Pin_3)
- net GPIO26: now reaches J1.37 (GPIO26)
- net GPIO26: now also J9.4 (Pin_4)
- net ~{RST}: now reaches J4.16 (Pin_2)
- net ~{RST}: now also J9.5 (Pin_5)
Other:
- note added: "ID EEPROM"
- note added: "Test Points"
- note removed: "ID EEPROM - CAT24C512"
- moved on the sheet: C1, C2, C3, C4, C5, C6, C7, C8, C9, D2, D3, D4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
