File: Hardware/SparkFun_GNSS_pHAT.kicad_sch (KiCad schematic)
At the start: 85 parts, among them J1 Raspberry_Pi_2x20_SMD_Passthr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, J2 Conn_02x10, J3 U.FL, J4 Conn_02x10, J5 microSD_Friction, J6 USB_C_Receptacle, J7 SMA_Edge, J8 Qwiic_Vertical, J9 Conn_01x05, U1 CAT24C512WI-GT3, U2 AP7361C-3.3V, U3 STLQ015-3.3

Commit message: pHAT updated after review
Parts:
- removed R14: 1k, SparkFun-Resistor:R_0603_1608Metric, symbol SparkFun-Resistor:1k_0603
- removed U3: STLQ015-3.3, SparkFun-Semiconductor-Standard:SOT23-5, symbol SparkFun-Regulator:STLQ015-3.3
- added R14: 4.7k, SparkFun-Resistor:R_0603_1608Metric, symbol SparkFun-Resistor:4.7k_0603
- added TP1, TP10, TP11, TP12, TP13, TP14, TP15, TP16, TP17, TP18, TP19, TP2, TP20, TP21, TP22, TP23, TP24, TP25, TP26, TP27, TP28, TP29, TP3, TP30, TP31, TP4, TP5, TP6, TP7, TP8, TP9: 1.25mm, SparkFun-Connector:TestPoint-1.25mm, symbol SparkFun-Connector:TestPoint_1.25mm
- added U3: RT9080-3.3, SparkFun-Semiconductor-Standard:SOT23-5, symbol SparkFun-Regulator:RT9080-3.3
- renumbered JP16 to JP10, JP17 to JP11, JP18 to JP12, JP19 to JP13, JP4 to JP14, JP5 to JP15, JP6 to JP22, JP7 to JP23, JP8 to JP24, JP9 to JP25, JP10 to JP4, JP11 to JP5, JP12 to JP6, JP13 to JP7, JP14 to JP8, JP15 to JP9, JP22 to PPS1.1, JP21 to PVT.1, JP23 to PWR.1, JP20 to RTK.1
Connections:
- net 5V: now also TP22.1, U3.1 (VIN), U3.3 (EN)
- net D+: now also TP25.1
- net D-: now also TP24.1
- net GND: now also TP31.1, U3.2 (GND)
- net ID_SC: now also TP2.1
- net ID_SD: now also TP1.1
- net Pi_3V3: now also TP23.1
- net SCL: now also TP4.1
- net SDA: now also TP3.1
- net SD_CLK: now also TP29.1
- net SD_CMD: now also TP30.1
- net SD_DAT0: now also TP28.1
- net SD_DAT3: now also TP27.1
- net VBACKUP: now also TP21.1, U3.5 (VOUT)
- net VUSB: now also TP26.1
- net at J1.29 (GCLK1/GPIO5), JP5.1 (A): now also TP6.1
- net at J1.33 (PWM1/GPIO13), JP13.1 (A): now also TP14.1
- net at J1.32 (PWM0/GPIO12), JP12.1 (A): now also TP13.1
- net at J1.22 (GPIO25), JP25.2 (B): now also TP20.1
- net at J1.23 (SCLK0/GPIO11), JP11.1 (A): now also TP12.1
- net at J1.26 (~{CE1}/GPIO7), JP7.1 (A): now also TP8.1
- net at J1.19 (PICO0/GPIO10), JP10.1 (A): now also TP11.1
- net at J1.31 (GCLK2/GPIO6), JP6.1 (A): now also TP7.1
- net at J1.18 (GPIO24), JP24.2 (B): now also TP19.1
- net at J1.24 (~{CE0}/GPIO8), JP8.1 (A): now also TP9.1
- net at J1.21 (POCI0/GPIO9), JP9.1 (A): now also TP10.1
- net at J1.7 (GCLK0/GPIO4), JP4.1 (A): now also TP5.1
- net at D6.2 (A): now also R14.2
- net at PWR.1.1 (A): now also R14.1
- net at J1.15 (GPIO22), JP22.2 (B): now also TP17.1
- net at J1.10 (GPIO15/RXD), JP15.2 (B): now also TP16.1
- net at J1.8 (GPIO14/TXD), JP14.2 (B): now also TP15.1
- net at J1.16 (GPIO23), JP23.2 (B): now also TP18.1
Other:
- note added: "I²C"
- note removed: "I2C"
- moved on the sheet: C10, C11, C12, C13, C14, C15, J1, J2, J4, J8, JP1, JP10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

Commit message: Update standoffs. Change panel to 2x2
Parts:
- J8: footprint SparkFun-Connector:JST_SMD_1.0mm-4_Vertical -> SparkFun-Connector:JST_SMD_1.0mm-4_Vertical_Black
- ST5, ST6, ST7, ST8: footprint SparkFun-Hardware:Standoff_Raspberry-Pi_HAT+ -> SparkFun-Hardware:Standoff_Hole-2.75mm_Clearance-1.625mm; symbol SparkFun-Hardware:Standoff_Raspberry-Pi_HAT+ -> SparkFun-Hardware:Standoff_Hole-2.75mm_Clearance-1.625mm; now left out of the parts list
Changed lines of the file:
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@@
 	)
 	(symbol
-		(lib_id "SparkFun-Hardware:Standoff_Raspberry-Pi_HAT+")
+		(lib_id "SparkFun-Hardware:Standoff_Hole-2.75mm_Clearance-1.625mm")
 		(at 243.84 175.26 0)
 		(unit 1)
 		(exclude_from_sim no)
-		(in_bom yes)
+		(in_bom no)
 		(on_board yes)
 		(dnp no)
@@
 			)
 		)
-		(property "Footprint" "SparkFun-Hardware:Standoff_Raspberry-Pi_HAT+"
+		(property "Footprint" "SparkFun-Hardware:Standoff_Hole-2.75mm_Clearance-1.625mm"
 			(at 243.84 182.88 0)
 			(effects
@@
 			)
 		)
-		(property "Footprint" "SparkFun-Connector:JST_SMD_1.0mm-4_Vertical"
+		(property "Footprint" "SparkFun-Connector:JST_SMD_1.0mm-4_Vertical_Black"
 			(at 246.38 85.09 0)
 			(effects
@@
 	)
 	(symbol
-		(lib_id "SparkFun-Hardware:Standoff_Raspberry-Pi_HAT+")
+		(lib_id "SparkFun-Hardware:Standoff_Hole-2.75mm_Clearance-1.625mm")
 		(at 243.84 179.07 0)
 		(unit 1)
 		(exclude_from_sim no)
-		(in_bom yes)
+		(in_bom no)
 		(on_board yes)
 		(dnp no)
@@
 			)
 		)
-		(property "Footprint" "SparkFun-Hardware:Standoff_Raspberry-Pi_HAT+"
+		(property "Footprint" "SparkFun-Hardware:Standoff_Hole-2.75mm_Clearance-1.625mm"
 			(at 243.84 186.69 0)
 			(effects
@@
 			)
 		)
-		(property "Description" "BF030-20A-B1-0360-0277-0600-LB 2x10 2.0mm Header"
+		(property "Description" "2x10 2.0mm Header with pegs"
 			(at 142.24 62.23 0)
 			(effects
@@
 			)
 		)
-		(property "Description" "BF030-20A-B1-0360-0277-0600-LB 2x10 2.0mm Header"
+		(property "Description" "2x10 2.0mm Header with pegs"
 			(at 200.66 62.23 0)
 			(effects
@@
 	)
 	(symbol
-		(lib_id "SparkFun-Hardware:Standoff_Raspberry-Pi_HAT+")
+		(lib_id "SparkFun-Hardware:Standoff_Hole-2.75mm_Clearance-1.625mm")
 		(at 247.65 179.07 0)
 		(unit 1)
 		(exclude_from_sim no)
-		(in_bom yes)
+		(in_bom no)
 		(on_board yes)
 		(dnp no)
@@
 			)
 		)
-		(property "Footprint" "SparkFun-Hardware:Standoff_Raspberry-Pi_HAT+"
+		(property "Footprint" "SparkFun-Hardware:Standoff_Hole-2.75mm_Clearance-1.625mm"
 			(at 247.65 186.69 0)
 			(effects
@@
 			)
 		)
-		(property "Description" "Generic connector, single row, 01x05, script generated (kicad-library-utils/schlib/autogen/connector/)"
+		(property "Description" "Basic 0.1\" PTH"
 			(at 90.17 102.87 0)
 			(effects
@@
 	)
 	(symbol
-		(lib_id "SparkFun-Hardware:Standoff_Raspberry-Pi_HAT+")
+		(lib_id "SparkFun-Hardware:Standoff_Hole-2.75mm_Clearance-1.625mm")
 		(at 247.65 175.26 0)
 		(unit 1)
 		(exclude_from_sim no)
-		(in_bom yes)
+		(in_bom no)
 		(on_board yes)
 		(dnp no)
@@
 			)
 		)
-		(property "Footprint" "SparkFun-Hardware:Standoff_Raspberry-Pi_HAT+"
+		(property "Footprint" "SparkFun-Hardware:Standoff_Hole-2.75mm_Clearance-1.625mm"
 			(at 247.65 182.88 0)
 			(effects

Commit message: Update RPi passthrough connector PROD_ID
Parts:
- J1: PROD_ID CONN-24972 -> CONN-13790
Changed lines of the file:
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@@
 	(title_block
 		(title "SparkFun GNSS pHAT")
-		(date "2025-01-29")
+		(date "2025-01-31")
 		(rev "v01")
 		(company "SparkFun")
@@
 			)
 		)
-		(property "Datasheet" "https://cdn.harwin.com/pdfs/M20-781.pdf"
+		(property "Datasheet" "http://www.4uconnector.com/online/object/4udrawing/10956.pdf"
 			(at 59.69 88.9 0)
 			(effects
@@
 			)
 		)
-		(property "PROD_ID" "CONN-24972"
+		(property "PROD_ID" "CONN-13790"
 			(at 59.69 96.52 0)
 			(effects

Commit message: Change I2C pull-ups to 3.9K RES-08701
Parts:
- R1, R2, R4, R5: value 3.6k -> 3.9k; symbol SparkFun-Resistor:3.6k_0603 -> SparkFun-Resistor:3.9k_0603; PROD_ID RES-08417 -> RES-08701
Other:
- moved on the sheet: R2, R4
Changed lines of the file:
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@@
 	)
 	(symbol
-		(lib_id "SparkFun-Resistor:3.6k_0603")
+		(lib_id "SparkFun-Resistor:3.9k_0603")
 		(at 251.46 54.61 90)
 		(unit 1)
@@
 			)
 		)
-		(property "Value" "3.6k"
+		(property "Value" "3.9k"
 			(at 254 55.8799 90)
 			(effects
@@
 			)
 		)
-		(property "PROD_ID" "RES-08417"
+		(property "PROD_ID" "RES-08701"
 			(at 258.318 54.61 0)
 			(effects
@@
 	)
 	(symbol
-		(lib_id "SparkFun-Resistor:3.6k_0603")
+		(lib_id "SparkFun-Resistor:3.9k_0603")
 		(at 251.46 35.56 90)
 		(unit 1)
@@
 			)
 		)
-		(property "Value" "3.6k"
+		(property "Value" "3.9k"
 			(at 254 36.8299 90)
 			(effects
@@
 			)
 		)
-		(property "PROD_ID" "RES-08417"
+		(property "PROD_ID" "RES-08701"
 			(at 258.318 35.56 0)
 			(effects
@@
 	)
 	(symbol
-		(lib_id "SparkFun-Resistor:3.6k_0603")
-		(at 243.84 35.56 270)
-		(mirror x)
+		(lib_id "SparkFun-Resistor:3.9k_0603")
+		(at 243.84 35.56 90)
 		(unit 1)
 		(exclude_from_sim no)
@@
 		(dnp no)
 		(property "Reference" "R4"
-			(at 238.76 34.29 90)
+			(at 241.3 34.2899 90)
 			(effects
 				(font
@@
 			)
 		)
-		(property "Value" "3.6k"
-			(at 237.49 36.83 90)
+		(property "Value" "3.9k"
+			(at 241.3 36.8299 90)
 			(effects
 				(font
@@
 		)
 		(property "Footprint" "SparkFun-Resistor:R_0603_1608Metric"
-			(at 239.268 35.56 0)
+			(at 248.412 35.56 0)
 			(effects
 				(font
@@
 		)
 		(property "Datasheet" "https://www.vishay.com/docs/20035/dcrcwe3.pdf"
-			(at 234.95 36.83 0)
+			(at 252.73 36.83 0)
 			(effects
 				(font
@@
 		)
 		(property "Description" "Resistor"
-			(at 232.41 35.56 0)
+			(at 255.27 35.56 0)
 			(effects
 				(font
@@
 			)
 		)
-		(property "PROD_ID" "RES-08417"
-			(at 236.982 35.56 0)
+		(property "PROD_ID" "RES-08701"
+			(at 250.698 35.56 0)
 			(effects
 				(font
@@
 	)
 	(symbol
-		(lib_id "SparkFun-Resistor:3.6k_0603")
-		(at 243.84 54.61 270)
-		(mirror x)
+		(lib_id "SparkFun-Resistor:3.9k_0603")
+		(at 243.84 54.61 90)
 		(unit 1)
 		(exclude_from_sim no)
@@
 		(dnp no)
 		(property "Reference" "R2"
-			(at 238.76 53.34 90)
+			(at 241.3 53.3399 90)
 			(effects
 				(font
@@
 			)
 		)
-		(property "Value" "3.6k"
-			(at 237.49 55.88 90)
+		(property "Value" "3.9k"
+			(at 241.3 55.8799 90)
 			(effects
 				(font
@@
 		)
 		(property "Footprint" "SparkFun-Resistor:R_0603_1608Metric"
-			(at 239.268 54.61 0)
+			(at 248.412 54.61 0)
 			(effects
 				(font
@@
 		)
 		(property "Datasheet" "https://www.vishay.com/docs/20035/dcrcwe3.pdf"
-			(at 234.95 55.88 0)
+			(at 252.73 55.88 0)
 			(effects
 				(font
@@
 		)
 		(property "Description" "Resistor"
-			(at 232.41 54.61 0)
+			(at 255.27 54.61 0)
 			(effects
 				(font
@@
 			)
 		)
-		(property "PROD_ID" "RES-08417"
-			(at 236.982 54.61 0)
+		(property "PROD_ID" "RES-08701"
+			(at 250.698 54.61 0)
 			(effects
 				(font

Commit message: v10 - update connectors and silk
Parts:
- J2, J4: footprint SparkFun-Connector:2x10_2.0mm_Male_Pins_Vertical_SMD -> SparkFun-Connector:2x10_2.0mm_Male_Pins_Vertical_SMD_Pegs; PROD_ID CONN-22476 -> CONN-25207
Connections:
- no-connect marks 0 -> 15
Other:
- note added: "Open jumpers to disable LEDs"
- note added: "Open jumpers to isolate GPIO pins"
- company: SparkFun -> SparkFun Electronics
- title: SparkFun GNSS pHAT -> SparkFun GNSS Flex pHAT
Changed lines of the file:
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@@
 	(paper "USLetter")
 	(title_block
-		(title "SparkFun GNSS pHAT")
-		(date "2025-01-31")
-		(rev "v01")
-		(company "SparkFun")
+		(title "SparkFun GNSS Flex pHAT")
+		(date "2025-03-20")
+		(rev "v10")
+		(company "SparkFun Electronics")
 		(comment 1 "Designed by: P.C.")
 	)
@@
 		(color 0 0 0 0)
 	)
+	(no_connect
+		(at 39.37 43.18)
+	)
+	(no_connect
+		(at 39.37 53.34)
+	)
+	(no_connect
+		(at 72.39 185.42)
+	)
+	(no_connect
+		(at 72.39 172.72)
+	)
+	(no_connect
+		(at 39.37 48.26)
+	)
+	(no_connect
+		(at 256.54 105.41)
+	)
+	(no_connect
+		(at 214.63 29.21)
+	)
+	(no_connect
+		(at 214.63 44.45)
+	)
+	(no_connect
+		(at 39.37 38.1)
+	)
+	(no_connect
+		(at 39.37 40.64)
+	)
+	(no_connect
+		(at 39.37 71.12)
+	)
+	(no_connect
+		(at 39.37 50.8)
+	)
+	(no_connect
+		(at 256.54 118.11)
+	)
+	(no_connect
+		(at 72.39 175.26)
+	)
+	(no_connect
+		(at 186.69 49.53)
+	)
 	(wire
 		(pts
@@
 		)
 	)
+	(text "Open jumpers to\ndisable LEDs"
+		(exclude_from_sim no)
+		(at 170.18 161.29 0)
+		(effects
+			(font
+				(size 1.016 1.016)
+			)
+		)
+	)
 	(text "Dielectric thickness (layer 1 to 2): 0.2mm"
 		(exclude_from_sim no)
@@
 		)
 	)
+	(text "Open jumpers to\nisolate GPIO pins"
+		(exclude_from_sim no)
+		(at 30.48 36.83 0)
+		(effects
+			(font
+				(size 1.016 1.016)
+			)
+		)
+	)
 	(text "ID EEPROM"
 		(exclude_from_sim no)
@@
 			)
 		)
-		(property "Footprint" "SparkFun-Connector:2x10_2.0mm_Male_Pins_Vertical_SMD"
+		(property "Footprint" "SparkFun-Connector:2x10_2.0mm_Male_Pins_Vertical_SMD_Pegs"
 			(at 142.24 57.15 0)
 			(effects
@@
 			)
 		)
-		(property "Datasheet" "https://gct.co/files/drawings/bf030.pdf"
+		(property "Datasheet" "http://www.4uconnector.com/online/object/4udrawing/22817.pdf"
 			(at 142.24 59.69 0)
 			(effects
@@
 			)
 		)
-		(property "PROD_ID" "CONN-22476"
+		(property "PROD_ID" "CONN-25207"
 			(at 142.24 64.77 0)
 			(effects
@@
 			)
 		)
-		(property "Footprint" "SparkFun-Connector:2x10_2.0mm_Male_Pins_Vertical_SMD"
+		(property "Footprint" "SparkFun-Connector:2x10_2.0mm_Male_Pins_Vertical_SMD_Pegs"
 			(at 200.66 57.15 0)
 			(effects
@@
 			)
 		)
-		(property "Datasheet" "https://gct.co/files/drawings/bf030.pdf"
+		(property "Datasheet" "http://www.4uconnector.com/online/object/4udrawing/22817.pdf"
 			(at 200.66 59.69 0)
 			(effects
@@
 			)
 		)
-		(property "PROD_ID" "CONN-22476"
+		(property "PROD_ID" "CONN-25207"
 			(at 200.66 64.77 0)
 			(effects
